File: level-shifter.kicad_sch (KiCad schematic)
At the start: 2 parts, among them U14 SN74LV1T125DBV

Commit message: schem: add sheet titles
Other:
- title: RPI CAN FD Power Hat+ -> S6TM Detect Carrier 2
Changed lines of the file:
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@@
 	(paper "A4")
 	(title_block
-		(title "RPI CAN FD Power Hat+")
-		(date "2026-04-11")
+		(title "S6TM Detect Carrier 2")
+		(date "2026-09-24")
 		(rev "01")
 		(company "Rémi Ait-Younes")

Commit message: schem: reannotate
Parts:
- renumbered C48 to C51, U14 to U15
Changed lines of the file:
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@@
 		(dnp no)
 		(fields_autoplaced yes)
-		(property "Reference" "#PWR0101"
+		(property "Reference" "#PWR0123"
 			(at 135.89 111.76 0)
 			(hide yes)
@@
 			(project "s6tm-detect-cb-2"
 				(path "/f4a18219-a653-4da9-9eb6-662d05c28432/2e4c8b7c-4e07-4d89-a615-6ea5caa4da61/32c3d493-1b0e-47fa-8917-a660b5c090e8"
-					(reference "#PWR0101")
+					(reference "#PWR0123")
 					(unit 1)
 				)
 				(path "/f4a18219-a653-4da9-9eb6-662d05c28432/2e4c8b7c-4e07-4d89-a615-6ea5caa4da61/385bdec9-6424-4b07-b543-e3b10735eeaa"
-					(reference "#PWR0114")
+					(reference "#PWR0132")
 					(unit 1)
 				)
 				(path "/f4a18219-a653-4da9-9eb6-662d05c28432/2e4c8b7c-4e07-4d89-a615-6ea5caa4da61/98ab9a83-ee49-418b-b983-049784f7f53f"
-					(reference "#PWR0106")
+					(reference "#PWR0126")
 					(unit 1)
 				)
 				(path "/f4a18219-a653-4da9-9eb6-662d05c28432/2e4c8b7c-4e07-4d89-a615-6ea5caa4da61/db2ef6a9-111c-4bec-afa1-ab77dd998347"
-					(reference "#PWR0110")
+					(reference "#PWR0129")
 					(unit 1)
 				)
 				(path "/f4a18219-a653-4da9-9eb6-662d05c28432/2e4c8b7c-4e07-4d89-a615-6ea5caa4da61/ddb8cfb5-d471-481d-b043-497a11b3c6cd"
-					(reference "#PWR0118")
+					(reference "#PWR0135")
 					(unit 1)
 				)
@@
 		(in_pos_files yes)
 		(dnp no)
-		(property "Reference" "C48"
+		(property "Reference" "C51"
 			(at 142.494 80.264 90)
 			(show_name no)
@@
 			(project "s6tm-detect-cb-2"
 				(path "/f4a18219-a653-4da9-9eb6-662d05c28432/2e4c8b7c-4e07-4d89-a615-6ea5caa4da61/32c3d493-1b0e-47fa-8917-a660b5c090e8"
-					(reference "C48")
+					(reference "C51")
 					(unit 1)
 				)
 				(path "/f4a18219-a653-4da9-9eb6-662d05c28432/2e4c8b7c-4e07-4d89-a615-6ea5caa4da61/385bdec9-6424-4b07-b543-e3b10735eeaa"
-					(reference "C51")
+					(reference "C54")
 					(unit 1)
 				)
 				(path "/f4a18219-a653-4da9-9eb6-662d05c28432/2e4c8b7c-4e07-4d89-a615-6ea5caa4da61/98ab9a83-ee49-418b-b983-049784f7f53f"
-					(reference "C49")
+					(reference "C52")
 					(unit 1)
 				)
 				(path "/f4a18219-a653-4da9-9eb6-662d05c28432/2e4c8b7c-4e07-4d89-a615-6ea5caa4da61/db2ef6a9-111c-4bec-afa1-ab77dd998347"
-					(reference "C50")
+					(reference "C53")
 					(unit 1)
 				)
 				(path "/f4a18219-a653-4da9-9eb6-662d05c28432/2e4c8b7c-4e07-4d89-a615-6ea5caa4da61/ddb8cfb5-d471-481d-b043-497a11b3c6cd"
-					(reference "C52")
+					(reference "C55")
 					(unit 1)
 				)
@@
 		(dnp no)
 		(fields_autoplaced yes)
-		(property "Reference" "#PWR0100"
+		(property "Reference" "#PWR0122"
 			(at 120.65 101.6 0)
 			(hide yes)
@@
 			(project "s6tm-detect-cb-2"
 				(path "/f4a18219-a653-4da9-9eb6-662d05c28432/2e4c8b7c-4e07-4d89-a615-6ea5caa4da61/32c3d493-1b0e-47fa-8917-a660b5c090e8"
-					(reference "#PWR0100")
+					(reference "#PWR0122")
 					(unit 1)
 				)
 				(path "/f4a18219-a653-4da9-9eb6-662d05c28432/2e4c8b7c-4e07-4d89-a615-6ea5caa4da61/385bdec9-6424-4b07-b543-e3b10735eeaa"
-					(reference "#PWR0113")
+					(reference "#PWR0131")
 					(unit 1)
 				)
 				(path "/f4a18219-a653-4da9-9eb6-662d05c28432/2e4c8b7c-4e07-4d89-a615-6ea5caa4da61/98ab9a83-ee49-418b-b983-049784f7f53f"
-					(reference "#PWR0105")
+					(reference "#PWR0125")
 					(unit 1)
 				)
 				(path "/f4a18219-a653-4da9-9eb6-662d05c28432/2e4c8b7c-4e07-4d89-a615-6ea5caa4da61/db2ef6a9-111c-4bec-afa1-ab77dd998347"
-					(reference "#PWR0109")
+					(reference "#PWR0128")
 					(unit 1)
 				)
 				(path "/f4a18219-a653-4da9-9eb6-662d05c28432/2e4c8b7c-4e07-4d89-a615-6ea5caa4da61/ddb8cfb5-d471-481d-b043-497a11b3c6cd"
-					(reference "#PWR0117")
+					(reference "#PWR0134")
 					(unit 1)
 				)
@@
 		(in_pos_files yes)
 		(dnp no)
-		(property "Reference" "U14"
+		(property "Reference" "U15"
 			(at 145.288 101.346 0)
 			(show_name no)
@@
 			(project "s6tm-detect-cb-2"
 				(path "/f4a18219-a653-4da9-9eb6-662d05c28432/2e4c8b7c-4e07-4d89-a615-6ea5caa4da61/32c3d493-1b0e-47fa-8917-a660b5c090e8"
-					(reference "U14")
+					(reference "U15")
 					(unit 1)
 				)
 				(path "/f4a18219-a653-4da9-9eb6-662d05c28432/2e4c8b7c-4e07-4d89-a615-6ea5caa4da61/385bdec9-6424-4b07-b543-e3b10735eeaa"
+					(reference "U18")
+					(unit 1)
+				)
+				(path "/f4a18219-a653-4da9-9eb6-662d05c28432/2e4c8b7c-4e07-4d89-a615-6ea5caa4da61/98ab9a83-ee49-418b-b983-049784f7f53f"
+					(reference "U16")
+					(unit 1)
+				)
+				(path "/f4a18219-a653-4da9-9eb6-662d05c28432/2e4c8b7c-4e07-4d89-a615-6ea5caa4da61/db2ef6a9-111c-4bec-afa1-ab77dd998347"
 					(reference "U17")
 					(unit 1)
 				)
-				(path "/f4a18219-a653-4da9-9eb6-662d05c28432/2e4c8b7c-4e07-4d89-a615-6ea5caa4da61/98ab9a83-ee49-418b-b983-049784f7f53f"
-					(reference "U15")
-					(unit 1)
-				)
-				(path "/f4a18219-a653-4da9-9eb6-662d05c28432/2e4c8b7c-4e07-4d89-a615-6ea5caa4da61/db2ef6a9-111c-4bec-afa1-ab77dd998347"
-					(reference "U16")
-					(unit 1)
-				)
 				(path "/f4a18219-a653-4da9-9eb6-662d05c28432/2e4c8b7c-4e07-4d89-a615-6ea5caa4da61/ddb8cfb5-d471-481d-b043-497a11b3c6cd"
-					(reference "U18")
+					(reference "U19")
 					(unit 1)
 				)
@@
 		(dnp no)
 		(fields_autoplaced yes)
-		(property "Reference" "#PWR0102"
+		(property "Reference" "#PWR0124"
 			(at 146.05 93.98 0)
 			(hide yes)
@@
 			(project "s6tm-detect-cb-2"
 				(path "/f4a18219-a653-4da9-9eb6-662d05c28432/2e4c8b7c-4e07-4d89-a615-6ea5caa4da61/32c3d493-1b0e-47fa-8917-a660b5c090e8"
-					(reference "#PWR0102")
+					(reference "#PWR0124")
 					(unit 1)
 				)
 				(path "/f4a18219-a653-4da9-9eb6-662d05c28432/2e4c8b7c-4e07-4d89-a615-6ea5caa4da61/385bdec9-6424-4b07-b543-e3b10735eeaa"
-					(reference "#PWR0115")
+					(reference "#PWR0133")
 					(unit 1)
 				)
 				(path "/f4a18219-a653-4da9-9eb6-662d05c28432/2e4c8b7c-4e07-4d89-a615-6ea5caa4da61/98ab9a83-ee49-418b-b983-049784f7f53f"
-					(reference "#PWR0107")
+					(reference "#PWR0127")
 					(unit 1)
 				)
 				(path "/f4a18219-a653-4da9-9eb6-662d05c28432/2e4c8b7c-4e07-4d89-a615-6ea5caa4da61/db2ef6a9-111c-4bec-afa1-ab77dd998347"
-					(reference "#PWR0111")
+					(reference "#PWR0130")
 					(unit 1)
 				)
 				(path "/f4a18219-a653-4da9-9eb6-662d05c28432/2e4c8b7c-4e07-4d89-a615-6ea5caa4da61/ddb8cfb5-d471-481d-b043-497a11b3c6cd"
-					(reference "#PWR0119")
-					(unit 1)
-				)
+					(reference "#PWR0136")
+					(unit 1)
+				)
