File: efuse.kicad_sch (KiCad schematic)
At the start: 12 parts, among them U9 TPS259472A

Commit message: schem: add sheet titles
Other:
- company: (none) -> Rémi Ait-Younes
- title: (none) -> S6TM Detect Carrier 2
Changed lines of the file:
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@@
 	(generator_version "10.0")
 	(paper "A4")
+	(title_block
+		(title "S6TM Detect Carrier 2")
+		(date "2026-09-24")
+		(rev "01")
+		(company "Rémi Ait-Younes")
+	)
 	(text "TPS259472A\n5A efuse"
 		(exclude_from_sim no)

Commit message: schem: reannotate
Parts:
- renumbered C22 to C36, C24 to C37, C23 to C38, C25 to C39, D5 to D9, R1 to R22, R13 to R23, R10 to R24, R11 to R25, R12 to R26, R2 to R27, U9 to U12
Changed lines of the file:
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@@
 		(dnp no)
 		(fields_autoplaced yes)
-		(property "Reference" "#PWR034"
+		(property "Reference" "#PWR087"
 			(at 135.89 100.33 0)
 			(hide yes)
@@
 			(project "s6tm-detect-cb-2"
 				(path "/f4a18219-a653-4da9-9eb6-662d05c28432/169cf3bf-dcdd-445b-abbd-86da239eca7a/7554ad60-3936-47eb-9d6b-43a6f6ab1674"
-					(reference "#PWR034")
+					(reference "#PWR087")
 					(unit 1)
 				)
@@
 		(dnp no)
 		(fields_autoplaced yes)
-		(property "Reference" "R12"
+		(property "Reference" "R26"
 			(at 170.18 83.8199 0)
 			(show_name no)
@@
 			(project "s6tm-detect-cb-2"
 				(path "/f4a18219-a653-4da9-9eb6-662d05c28432/169cf3bf-dcdd-445b-abbd-86da239eca7a/7554ad60-3936-47eb-9d6b-43a6f6ab1674"
-					(reference "R12")
+					(reference "R26")
 					(unit 1)
 				)
@@
 		(in_pos_files yes)
 		(dnp no)
-		(property "Reference" "R2"
+		(property "Reference" "R27"
 			(at 170.18 93.9799 0)
 			(show_name no)
@@
 			(project "s6tm-detect-cb-2"
 				(path "/f4a18219-a653-4da9-9eb6-662d05c28432/169cf3bf-dcdd-445b-abbd-86da239eca7a/7554ad60-3936-47eb-9d6b-43a6f6ab1674"
-					(reference "R2")
+					(reference "R27")
 					(unit 1)
 				)
@@
 		(dnp no)
 		(fields_autoplaced yes)
-		(property "Reference" "R10"
+		(property "Reference" "R24"
 			(at 146.05 111.76 90)
 			(show_name no)
@@
 			(project "s6tm-detect-cb-2"
 				(path "/f4a18219-a653-4da9-9eb6-662d05c28432/169cf3bf-dcdd-445b-abbd-86da239eca7a/7554ad60-3936-47eb-9d6b-43a6f6ab1674"
-					(reference "R10")
+					(reference "R24")
 					(unit 1)
 				)
@@
 		(dnp no)
 		(fields_autoplaced yes)
-		(property "Reference" "#PWR058"
+		(property "Reference" "#PWR092"
 			(at 184.15 100.33 0)
 			(hide yes)
@@
 			(project "s6tm-detect-cb-2"
 				(path "/f4a18219-a653-4da9-9eb6-662d05c28432/169cf3bf-dcdd-445b-abbd-86da239eca7a/7554ad60-3936-47eb-9d6b-43a6f6ab1674"
-					(reference "#PWR058")
+					(reference "#PWR092")
 					(unit 1)
 				)
@@
 		(in_pos_files yes)
 		(dnp no)
-		(property "Reference" "R13"
+		(property "Reference" "R23"
 			(at 129.54 93.9799 0)
 			(show_name no)
@@
 			(project "s6tm-detect-cb-2"
 				(path "/f4a18219-a653-4da9-9eb6-662d05c28432/169cf3bf-dcdd-445b-abbd-86da239eca7a/7554ad60-3936-47eb-9d6b-43a6f6ab1674"
-					(reference "R13")
+					(reference "R23")
 					(unit 1)
 				)
@@
 		(dnp no)
 		(fields_autoplaced yes)
-		(property "Reference" "#PWR045"
+		(property "Reference" "#PWR088"
 			(at 140.97 118.11 0)
 			(hide yes)
@@
 			(project "s6tm-detect-cb-2"
 				(path "/f4a18219-a653-4da9-9eb6-662d05c28432/169cf3bf-dcdd-445b-abbd-86da239eca7a/7554ad60-3936-47eb-9d6b-43a6f6ab1674"
-					(reference "#PWR045")
+					(reference "#PWR088")
 					(unit 1)
 				)
@@
 		(in_pos_files yes)
 		(dnp no)
-		(property "Reference" "C24"
+		(property "Reference" "C37"
 			(at 140.208 98.552 90)
 			(show_name no)
@@
 			(project "s6tm-detect-cb-2"
 				(path "/f4a18219-a653-4da9-9eb6-662d05c28432/169cf3bf-dcdd-445b-abbd-86da239eca7a/7554ad60-3936-47eb-9d6b-43a6f6ab1674"
-					(reference "C24")
+					(reference "C37")
 					(unit 1)
 				)
@@
 		(dnp no)
 		(fields_autoplaced yes)
-		(property "Reference" "#FLG06"
+		(property "Reference" "#FLG07"
 			(at 121.92 78.105 0)
 			(hide yes)
@@
 			(project "s6tm-detect-cb-2"
 				(path "/f4a18219-a653-4da9-9eb6-662d05c28432/169cf3bf-dcdd-445b-abbd-86da239eca7a/7554ad60-3936-47eb-9d6b-43a6f6ab1674"
-					(reference "#FLG06")
+					(reference "#FLG07")
 					(unit 1)
 				)
@@
 		(dnp no)
 		(fields_autoplaced yes)
-		(property "Reference" "#PWR054"
+		(property "Reference" "#PWR090"
 			(at 167.64 106.68 0)
 			(hide yes)
@@
 			(project "s6tm-detect-cb-2"
 				(path "/f4a18219-a653-4da9-9eb6-662d05c28432/169cf3bf-dcdd-445b-abbd-86da239eca7a/7554ad60-3936-47eb-9d6b-43a6f6ab1674"
-					(reference "#PWR054")
+					(reference "#PWR090")
 					(unit 1)
 				)
@@
 		(in_pos_files yes)
 		(dnp no)
-		(property "Reference" "C22"
+		(property "Reference" "C36"
 			(at 120.142 89.154 0)
 			(show_name no)
@@
 			(project "s6tm-detect-cb-2"
 				(path "/f4a18219-a653-4da9-9eb6-662d05c28432/169cf3bf-dcdd-445b-abbd-86da239eca7a/7554ad60-3936-47eb-9d6b-43a6f6ab1674"
-					(reference "C22")
+					(reference "C36")
 					(unit 1)
 				)
@@
 		(dnp no)
 		(fields_autoplaced yes)
-		(property "Reference" "#PWR048"
+		(property "Reference" "#PWR089"
 			(at 161.29 121.92 0)
 			(hide yes)
@@
 			(project "s6tm-detect-cb-2"
 				(path "/f4a18219-a653-4da9-9eb6-662d05c28432/169cf3bf-dcdd-445b-abbd-86da239eca7a/7554ad60-3936-47eb-9d6b-43a6f6ab1674"
-					(reference "#PWR048")
+					(reference "#PWR089")
 					(unit 1)
 				)
@@
 		(in_pos_files yes)
 		(dnp no)
-		(property "Reference" "C25"
+		(property "Reference" "C39"
 			(at 189.484 87.376 0)
 			(show_name no)
@@
 			(project "s6tm-detect-cb-2"
 				(path "/f4a18219-a653-4da9-9eb6-662d05c28432/169cf3bf-dcdd-445b-abbd-86da239eca7a/7554ad60-3936-47eb-9d6b-43a6f6ab1674"
-					(reference "C25")
+					(reference "C39")
 					(unit 1)
 				)
@@
 		(dnp no)
 		(fields_autoplaced yes)
-		(property "Reference" "#PWR09"
+		(property "Reference" "#PWR085"
 			(at 123.19 101.6 0)
 			(hide yes)
@@
 			(project "s6tm-detect-cb-2"
 				(path "/f4a18219-a653-4da9-9eb6-662d05c28432/169cf3bf-dcdd-445b-abbd-86da239eca7a/7554ad60-3936-47eb-9d6b-43a6f6ab1674"
-					(reference "#PWR09")
+					(reference "#PWR085")
 					(unit 1)
 				)
@@
 		(dnp no)
 		(fields_autoplaced yes)
-		(property "Reference" "#PWR032"
+		(property "Reference" "#PWR086"
 			(at 132.08 106.68 0)
 			(hide yes)
@@
 			(project "s6tm-detect-cb-2"
 				(path "/f4a18219-a653-4da9-9eb6-662d05c28432/169cf3bf-dcdd-445b-abbd-86da239eca7a/7554ad60-3936-47eb-9d6b-43a6f6ab1674"
-					(reference "#PWR032")
+					(reference "#PWR086")
 					(unit 1)
 				)
@@
 		(in_pos_files yes)
 		(dnp no)
-		(property "Reference" "C23"
+		(property "Reference" "C38"
 			(at 180.594 83.058 0)
 			(show_name no)
@@
 			(project "s6tm-detect-cb-2"
 				(path "/f4a18219-a653-4da9-9eb6-662d05c28432/169cf3bf-dcdd-445b-abbd-86da239eca7a/7554ad60-3936-47eb-9d6b-43a6f6ab1674"
-					(reference "C23")
+					(reference "C38")
 					(unit 1)
 				)
@@
 		(in_pos_files yes)
 		(dnp no)
-		(property "Reference" "#PWR055"
+		(property "Reference" "#PWR091"
 			(at 171.45 106.68 0)
 			(hide yes)
@@
 			(project "s6tm-detect-cb-2"
 				(path "/f4a18219-a653-4da9-9eb6-662d05c28432/169cf3bf-dcdd-445b-abbd-86da239eca7a/7554ad60-3936-47eb-9d6b-43a6f6ab1674"
-					(reference "#PWR055")
+					(reference "#PWR091")
 					(unit 1)
 				)
@@
 		(dnp no)
 		(fields_autoplaced yes)
-		(property "Reference" "U9"
+		(property "Reference" "U12"
 			(at 151.765 72.39 0)
 			(show_name no)
@@
 			(project "s6tm-detect-cb-2"
 				(path "/f4a18219-a653-4da9-9eb6-662d05c28432/169cf3bf-dcdd-445b-abbd-86da239eca7a/7554ad60-3936-47eb-9d6b-43a6f6ab1674"
-					(reference "U9")
+					(reference "U12")
 					(unit 1)
 				)
@@
 		(in_pos_files yes)
 		(dnp no)
-		(property "Reference" "D5"
+		(property "Reference" "D9"
 			(at 165.1 113.284 90)
 			(show_name no)
@@
 			(project "s6tm-detect-cb-2"
 				(path "/f4a18219-a653-4da9-9eb6-662d05c28432/169cf3bf-dcdd-445b-abbd-86da239eca7a/7554ad60-3936-47eb-9d6b-43a6f6ab1674"
-					(reference "D5")
+					(reference "D9")
 					(unit 1)
 				)
@@
 		(in_pos_files yes)
 		(dnp no)
-		(property "Reference" "R11"
+		(property "Reference" "R25"
 			(at 166.624 107.95 90)
 			(show_name no)
@@
 			(project "s6tm-detect-cb-2"
 				(path "/f4a18219-a653-4da9-9eb6-662d05c28432/169cf3bf-dcdd-445b-abbd-86da239eca7a/7554ad60-3936-47eb-9d6b-43a6f6ab1674"
-					(reference "R11")
+					(reference "R25")
 					(unit 1)
 				)
@@
 		(dnp no)
 		(fields_autoplaced yes)
-		(property "Reference" "R1"
+		(property "Reference" "R22"
 			(at 129.54 83.8199 0)
 			(show_name no)
@@
 			(project "s6tm-detect-cb-2"
 				(path "/f4a18219-a653-4da9-9eb6-662d05c28432/169cf3bf-dcdd-445b-abbd-86da239eca7a/7554ad60-3936-47eb-9d6b-43a6f6ab1674"
-					(reference "R1")
+					(reference "R22")
 					(unit 1)
 				)

Commit message: schem: update 10u caps to 0603
Parts:
- C38, C39: footprint Capacitor_SMD:C_0402_1005Metric -> Capacitor_SMD:C_0603_1608Metric; JLCPCB Part # C15525 -> C19702; Manufacturer Part Number CL05A106MQ5NUNC -> CL10A106KP8NNNC
Changed lines of the file:
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@@
 			)
 		)
-		(property "Footprint" "Capacitor_SMD:C_0402_1005Metric"
+		(property "Footprint" "Capacitor_SMD:C_0603_1608Metric"
 			(at 187.6552 91.44 0)
 			(hide yes)
@@
 			)
 		)
-		(property "JLCPCB Part #" "C15525"
+		(property "JLCPCB Part #" "C19702"
 			(at 186.69 87.63 0)
 			(hide yes)
@@
 			)
 		)
-		(property "Manufacturer Part Number" "CL05A106MQ5NUNC"
+		(property "Manufacturer Part Number" "CL10A106KP8NNNC"
 			(at 186.69 87.63 0)
 			(hide yes)
@@
 			)
 		)
-		(property "Footprint" "Capacitor_SMD:C_0402_1005Metric"
+		(property "Footprint" "Capacitor_SMD:C_0603_1608Metric"
 			(at 180.6448 91.44 0)
 			(hide yes)
@@
 			)
 		)
-		(property "JLCPCB Part #" "C15525"
+		(property "JLCPCB Part #" "C19702"
 			(at 181.61 87.63 0)
 			(hide yes)
@@
 			)
 		)
-		(property "Manufacturer Part Number" "CL05A106MQ5NUNC"
-			(at 181.61 87.63 0)
-			(hide yes)
+		(property "Manufacturer Part Number" "CL10A106KP8NNNC"
+			(at 181.61 87.63 0)
+			(hide yes)
